Commit message: SLAM, Nav, Launches & Meshs

File: description/robot.urdf.xacro (robot description, xacro)
@@ -1,187 +1,16 @@
 <?xml version="1.0"?>
-<robot xmlns:xacro="http://www.ros.org/wiki/xacro" name="autords">
-  <!--include xacro files from description files-->
-  <!-- <xacro:include filename="gazebo_control.xacro" /> -->
-  <xacro:include filename="ros2_control.xacro" />
-  <!-- Define materials -->
-  <material name="white">
-    <color rgba="1 1 1 1"/>
-  </material>
-  <material name="blue">
-    <color rgba="0.00784313725490196 0.23921568627451 0.823529411764706 1"/>
-  </material>
-  <material name="gray">
-    <color rgba="0.43921568627451 0.43921568627451 0.43921568627451 1"/>
-  </material>
-  <material name="green">
-    <color rgba="0 1 0 1"/>
-  </material>
-  <material name="red">
-    <color rgba="1 0 0 1"/>
-  </material>
-    <!-- Include inertial macros -->
-    <xacro:include filename="inertial_macros.xacro"/>
-  <!-- Define robot properties -->
-  <xacro:property name="radius" value="0.584"/>
-  <xacro:property name="height" value="0.663103892"/>
-  <!-- Define links -->
-  <link name="base_link">
-  </link>
- <joint name="base_footprint_joint" type="fixed">
-        <parent link="base_link"/>
-        <child link="base_footprint"/>
-        <origin xyz="0 0 0" rpy="0 0 0"/>
-    </joint>
-    <link name="base_footprint">
-    </link>
-  <link name="basefixed">
-    <visual>
-      <geometry>
-        <cylinder radius="${radius}" length="${height}"/>
-      </geometry>
-      <material name="white"/>
-    </visual>
-    <collision>
-      <geometry>
-        <cylinder radius="${radius}" length="${height}"/>
-      </geometry>
-    </collision>
-  </link>
-  <joint name="fixed" type="fixed">
-    <parent link="base_link"/>
-    <child link="basefixed"/>
-    <origin xyz="0 0 0.41549" rpy="0 0 0"/>
-  </joint>
-  <link name="right">
-    <visual>
-        <origin xyz="0.19 0.003997 -0.3902" rpy="1 0 0"/>
-      <geometry>
-        <cylinder radius="0.1" length="0.025"/>
-      </geometry>
-      <material name="blue"/>
-    </visual>
-    <collision>
-      <geometry>
-        <sphere radius="0.1"/>
-      </geometry>
-    </collision>
-  </link>
-  <joint name="right_wheel" type="continuous">
-    <parent link="basefixed"/>
-    <child link="right"/>
-    <origin xyz="0.19 0.003997 -0.3902" rpy="1 0 0"/>
-  </joint>
-  <link name="left">
-    <visual>
-        <origin xyz="-0.19 0.003997 -0.3902" rpy="1 0 0"/>
-      <geometry>
-        <cylinder radius="0.1" length="0.025"/>
-      </geometry>
-      <material name="blue"/>
-    </visual>
-    <collision>
-      <geometry>
-        <sphere radius="0.1"/>
-      </geometry>
-    </collision>
-  </link>
-  <joint name="left_wheel" type="continuous">
-    <parent link="basefixed"/>
-    <child link="left"/>
-    <origin xyz="-0.19 0.003997 -0.3902" rpy="1 0 0"/>
-  </joint>
-  <link name="front_free">
-    <visual>
-        <origin xyz="0 -0.17797 0.44185" rpy="0 0 0"/>
-      <geometry>
-        <sphere radius="0.022122419"/>
-      </geometry>
-      <material name="green"/>
-    </visual>
-    <collision>
-      <geometry>
-        <sphere radius="0.022122419"/>
-      </geometry>
-    </collision>
-  </link>
-  <joint name="front_free_joint" type="fixed">
-    <parent link="basefixed"/>
-    <child link="front_free"/>
-    <origin xyz="0 -0.17797 0.44185" rpy="0 0 0"/>
-  </joint>
-  <link name="back_free">
-    <visual>
-        <origin xyz="0 0.17783 0.44185" rpy="0 0 0"/>
-      <geometry>
-        <sphere radius="0.022122419"/>
-      </geometry>
-      <material name="green"/>
-    </visual>
-    <collision>
-      <geometry>
-        <sphere radius="0.022122419"/>
-      </geometry>
-    </collision>
-  </link>
-  <joint name="back_free_joint" type="fixed">
-    <parent link="basefixed"/>
-    <child link="back_free"/>
-    <origin xyz="0 0.17783 0.44185" rpy="0 0 0"/>
-  </joint>
-   <joint name="laser_joint" type="fixed">
-        <parent link="basefixed"/>
-        <child link="laser_frame"/>
-        <origin xyz="0.122 0 0.212" rpy="0 0 0"/>
-    </joint>
-    <link name="laser_frame">
-        <visual>
-            <geometry>
-                <cylinder radius="0.05" length="0.04"/>
-            </geometry>
-            <material name="black"/>
-        </visual>
-        <visual>
-            <origin xyz="0 0 -0.05"/>
-            <geometry>
-                <cylinder radius="0.01" length="0.1"/>
-            </geometry>
-            <material name="black"/>
-        </visual>
-        <collision>
-            <geometry>
-                <cylinder radius="0.05" length="0.04"/>
-            </geometry>
-        </collision>
-        <xacro:inertial_cylinder mass="0.1" length="0.04" radius="0.05">
-            <origin xyz="0 0 0" rpy="0 0 0"/>
-        </xacro:inertial_cylinder>
-    </link>
-    <gazebo reference="laser_frame">
-        <material>Gazebo/Black</material>
-        <sensor name="laser" type="ray">
-            <pose> 0 0 0 0 0 0 </pose>
-            <visualize>false</visualize>
-            <update_rate>10</update_rate>
-            <ray>
-                <scan>
-                    <horizontal>
-                        <samples>360</samples>
-                        <min_angle>-3.14</min_angle>
-                        <max_angle>3.14</max_angle>
-                    </horizontal>
-                </scan>
-                <range>
-                    <min>0.3</min>
-                    <max>12</max>
-                </range>
-            </ray>
-            <plugin name="laser_controller" filename="libgazebo_ros_ray_sensor.so">
-                <ros>
-                    <argument>~/out:=scan</argument>
-                </ros>
-                <output_type>sensor_msgs/LaserScan</output_type>
-                <frame_name>laser_frame</frame_name>
-            </plugin>
-        </sensor>
-    </gazebo>
+<robot xmlns:xacro="http://www.ros.org/wiki/xacro"  name="robot">
+    <xacro:arg name="use_ros2_control" default="true"/>
+    <xacro:arg name="sim_mode" default="false"/>
+    <xacro:include filename="robot_core.xacro" />
+    <xacro:if value="$(arg use_ros2_control)">
+        <xacro:include filename="ros2_control.xacro" />
+    </xacro:if>
+    <xacro:unless value="$(arg use_ros2_control)">
+        <xacro:include filename="gazebo_control.xacro" />
+    </xacro:unless>
+    <xacro:include filename="lidar.xacro" />
+    <!--xacro:include filename="camera.xacro" /-->
+    <!-- <xacro:include filename="depth_camera.xacro" /> -->
+    <!--xacro:include filename="face.xacro" /-->
 </robot>

File: description/ros2_control.xacro (robot description, xacro)
@@ -1,28 +1,61 @@
 <?xml version="1.0"?>
 <robot xmlns:xacro="http://www.ros.org/wiki/xacro">
-    <ros2_control name="GazeboSystem" type="system">
-        <hardware>
-            <plugin>gazebo_ros2_control/GazeboSystem</plugin>
-        </hardware>
-        <joint name="left_wheel">
-            <command_interface name="velocity">
-                <param name="min">-255</param>
-                <param name="max">255</param>
-            </command_interface>
-            <state_interface name="velocity"/>
-            <state_interface name="position"/>
-        </joint>
-        <joint name="right_wheel">
-            <command_interface name="velocity">
-                <param name="min">-255</param>
-                <param name="max">255</param>
-            </command_interface>
-            <state_interface name="velocity"/>
-            <state_interface name="position"/>
-        </joint>
-    </ros2_control>
+    <xacro:unless value="$(arg sim_mode)">
+        <ros2_control name="RealRobot" type="system">
+            <hardware>
+                <plugin>diffdrive_arduino/DiffDriveArduino</plugin>
+                <param name="left_wheel_name">left_wheel_joint</param>
+                <param name="right_wheel_name">right_wheel_joint</param>
+                <param name="loop_rate">30</param>
+                <param name="device">/dev/ttyUSB0</param>
+                <param name="baud_rate">57600</param>
+                <param name="timeout">1000</param>
+                <param name="enc_counts_per_rev">3436</param>
+            </hardware>
+            <joint name="left_wheel_joint">
+                <command_interface name="velocity">
+                    <param name="min">-10</param>
+                    <param name="max">10</param>
+                </command_interface>
+                <state_interface name="velocity"/>
+                <state_interface name="position"/>
+            </joint>
+            <joint name="right_wheel_joint">
+                <command_interface name="velocity">
+                    <param name="min">-10</param>
+                    <param name="max">10</param>
+                </command_interface>
+                <state_interface name="velocity"/>
+                <state_interface name="position"/>
+            </joint>
+        </ros2_control>
+    </xacro:unless>
+    <xacro:if value="$(arg sim_mode)">
+        <ros2_control name="GazeboSystem" type="system">
+            <hardware>
+                <plugin>gazebo_ros2_control/GazeboSystem</plugin>
+            </hardware>
+            <joint name="left_wheel_joint">
+                <command_interface name="velocity">
+                    <param name="min">-10</param>
+                    <param name="max">10</param>
+                </command_interface>
+                <state_interface name="velocity"/>
+                <state_interface name="position"/>
+            </joint>
+            <joint name="right_wheel_joint">
+                <command_interface name="velocity">
+                    <param name="min">-10</param>
+                    <param name="max">10</param>
+                </command_interface>
+                <state_interface name="velocity"/>
+                <state_interface name="position"/>
+            </joint>
+        </ros2_control>
+    </xacro:if>
     <gazebo>
         <plugin name="gazebo_ros2_control" filename="libgazebo_ros2_control.so">
-            <parameters>$(find autords)/config/my_controllers.yaml</parameters>
+            <parameters>$(find articubot_one)/config/my_controllers.yaml</parameters>
+            <parameters>$(find articubot_one)/config/gaz_ros2_ctl_use_sim.yaml</parameters>
         </plugin>
     </gazebo>
