Commit message: final test

File: description/gazebo_control.xacro (robot description, xacro)
@@ -6,6 +6,6 @@
             <left_joint>left_wheel_joint</left_joint>
             <right_joint>right_wheel_joint</right_joint>
-            <wheel_separation>0.297</wheel_separation>
-            <wheel_diameter>0.066</wheel_diameter>
+            <wheel_separation>0.34</wheel_separation>
+            <wheel_diameter>0.1</wheel_diameter>
             <!-- Limits -->
             <max_wheel_torque>200</max_wheel_torque>

File: description/lidar.xacro (robot description, xacro)
@@ -4,5 +4,5 @@
         <parent link="chassis"/>
         <child link="laser_frame"/>
-        <origin xyz="0 0 0.69645" rpy="0 0 0"/>
+        <origin xyz="0 0 0.663103892" rpy="0 0 0"/>
     </joint>
     <link name="laser_frame">
@@ -14,5 +14,5 @@
         </visual>
         <visual>
-            <origin xyz="0 0 -0.05"/>
+            <origin xyz="0 0 0"/>
             <geometry>
                 <cylinder radius="0.03471" length="0.01874"/>

File: description/robot.urdf.xacro (robot description, xacro)
@@ -11,6 +11,3 @@
     </xacro:unless>
     <xacro:include filename="lidar.xacro" />
-    <!--xacro:include filename="camera.xacro" /-->
-    <!-- <xacro:include filename="depth_camera.xacro" /> -->
-    <!--xacro:include filename="face.xacro" /-->
 </robot>

File: description/robot_core.xacro (robot description, xacro)
@@ -5,5 +5,5 @@
     <xacro:property name="chassis_height" value="0.663103892"/>
     <xacro:property name="chassis_mass" value="13.0"/>
-    <xacro:property name="wheel_radius" value="0.1"/>
+    <xacro:property name="wheel_radius" value="0.05"/>
     <xacro:property name="wheel_thickness" value="0.025"/>
     <xacro:property name="wheel_mass" value="0.2494"/>
@@ -11,8 +11,8 @@
     <xacro:property name="wheel_offset_y" value="0.165"/>
     <xacro:property name="wheel_offset_z" value="0.01"/>
-    <xacro:property name="caster_wheel_radius" value="0.022122419"/>
+    <xacro:property name="caster_wheel_radius" value="0.04"/>
     <xacro:property name="caster_wheel_mass" value="0.073417"/>
     <xacro:property name="caster_wheel_offset_x" value="0.1779"/>
-    <xacro:property name="caster_wheel_offset_z" value="0.005"/>
+    <xacro:property name="caster_wheel_offset_z" value="0"/>
     <material name="white">
         <color rgba="1 1 1 1" />
@@ -87,5 +87,5 @@
         <collision>
             <geometry>
-                <sphere radius="${wheel_radius}"/>
+                <cylinder radius="${wheel_radius}" length="${wheel_thickness}"/>
             </geometry>
         </collision>
@@ -113,5 +113,5 @@
         <collision>
             <geometry>
-                <sphere radius="${wheel_radius}"/>
+                <cylinder radius="${wheel_radius}" length="${wheel_thickness}"/>
             </geometry>
         </collision>
@@ -147,6 +147,6 @@
     <gazebo reference="caster_wheel_forward">
         <material>Gazebo/White</material>
-        <mu1 value="0.001"/>
-        <mu2 value="0.001"/>
+        <mu1 value="0.002"/>
+        <mu2 value="0.002"/>
     </gazebo>
    <!-- CASTER WHEEL LINK BACKWARD-->
@@ -172,8 +172,8 @@
         </xacro:inertial_sphere>
     </link>
-    <gazebo reference="caster_wheel">
+    <gazebo reference="caster_wheel_backward">
         <material>Gazebo/White</material>
-        <mu1 value="0.001"/>
-        <mu2 value="0.001"/>
+        <mu1 value="0.002"/>
+        <mu2 value="0.002"/>
     </gazebo>
 </robot>

File: description/ros2_control.xacro (robot description, xacro)
@@ -8,5 +8,5 @@
                 <param name="right_wheel_name">right_wheel_joint</param>
                 <param name="loop_rate">30</param>
-                <param name="device">/dev/ttyUSB0</param>
+                <param name="device">/dev/ttyACM0</param>
                 <param name="baud_rate">57600</param>
                 <param name="timeout">1000</param>
